Commit message: Fixed can not use moveit to control robot in Gazebo.

File: franka_panda_description/robots/panda_arm.xacro (robot description, xacro)
@@ -3,11 +3,4 @@
   <xacro:macro name="panda_arm" params="arm_id:='panda' description_pkg:='franka_panda_description' in_gazebo='' xyz:='0 0 0' rpy:='0 0 0'">
     <link name="world" />
-    <joint name="robot_to_world" type="fixed">
-      <parent link="world" />
-      <child link="${arm_id}_link0" />
-      <origin xyz="0.0 0.0 0.0" rpy="0.0 0.0 0.0" />
-      <axis xyz="0 0 1"/>
-      <dynamics damping="1.0"/>
-    </joint>
     <link name="${arm_id}_link0">
       <visual>
@@ -29,4 +22,11 @@
       </xacro:unless>
     </link>
+    <joint name="robot_to_world" type="fixed">
+      <parent link="world" />
+      <child link="${arm_id}_link0" />
+      <origin xyz="0.0 0.0 0.0" rpy="0.0 0.0 0.0" />
+      <axis xyz="0 0 1"/>
+      <dynamics damping="1.0"/>
+    </joint>
     <link name="${arm_id}_link1">
       <visual>

File: franka_panda_description/robots/panda_arm_hand.urdf.xacro (robot description, xacro)
@@ -4,5 +4,5 @@
   <xacro:arg name="load_gripper" default="true"/>
   <xacro:arg name="load_gazebo" default="true"/>
-  <xacro:arg name="use_gazebo_control" default="false"/>
+  <xacro:arg name="use_gazebo_control" default="true"/>
   <xacro:include filename="$(find franka_panda_description)/robots/panda_arm.xacro"/>
   <xacro:if value="$(arg load_gripper)">
