Commit message: Fixed joints on incoming goal don't match the controller joints and update panda_hand_controller pid gains.

File: franka_panda_description/robots/hand.xacro (robot description, xacro)
@@ -75,5 +75,4 @@
       <limit effort="20" lower="0.0" upper="0.04" velocity="0.2"/>
       <dynamics damping="500.0" friction="0.0"/>
-      <mimic joint="${ns}_finger_joint1" />
     </joint>
   </xacro:macro>
